Commit message: adding a sweeper geometry

File: description/robot.urdf.xacro (robot description, xacro)
@@ -7,4 +7,5 @@
     <xacro:include filename="materials.xacro"/>
     <xacro:include filename="robot_core.xacro"/>
+    <xacro:include filename="sweeper.xacro"/>
     <xacro:include filename="range_sensors.xacro"/>
     <xacro:include filename="lidar.xacro"/>

File: description/robot_core.xacro (robot description, xacro)
@@ -47,9 +47,9 @@
     <xacro:property name="wheel_color" value="blue"/>
     <xacro:property name="wheel_offset_x" value="0"/>
-    <xacro:property name="wheel_separatio" value="0.231"/>
+    <xacro:property name="wheel_separation" value="0.231"/>
     <joint name="left_wheel_joint" type="continuous">
         <parent link="base_link"/>
         <child link="left_wheel"/>
-        <origin xyz="${wheel_offset_x} ${wheel_separatio/2} ${wheel_radius}" rpy="-${pi/2} 0 0" />
+        <origin xyz="${wheel_offset_x} ${wheel_separation/2} ${wheel_radius}" rpy="-${pi/2} 0 0" />
         <axis xyz="0 0 1"/>
     </joint>
@@ -74,5 +74,5 @@
         <parent link="base_link"/>
         <child link="right_wheel"/>
-        <origin xyz="${wheel_offset_x} ${-wheel_separatio/2} ${wheel_radius}" rpy="${pi/2} 0 0" />
+        <origin xyz="${wheel_offset_x} ${-wheel_separation/2} ${wheel_radius}" rpy="${pi/2} 0 0" />
         <axis xyz="0 0 -1"/>
     </joint>
