Commit message: changing lidar orientation for real robot

File: description/lidar.xacro (robot description, xacro)
@@ -10,5 +10,10 @@
         <parent link="chassis"/>
         <child link="lidar_frame"/>
-        <origin xyz="0 0 ${chassis_thickness/2 + lidar_offset_z}" rpy="0 0 0"/>
+        <xacro:if value="$(arg sim_mode)">
+            <origin xyz="0 0 ${chassis_thickness/2 + lidar_offset_z}" rpy="0 0 0"/>
+        </xacro:if>
+        <xacro:unless value="$(arg sim_mode)">
+            <origin xyz="0 0 ${chassis_thickness/2 + lidar_offset_z}" rpy="0 0 ${pi}"/>
+        </xacro:unless>
     </joint>
     <link name="lidar_frame">

Commit message: adding lidar sensor STL files to URDF

File: description/lidar.xacro (robot description, xacro)
@@ -1,62 +1,112 @@
 <?xml version="1.0"?>
 <robot xmlns:xacro="http://www.ros.org/wiki/xacro" >
-    <!-- Lidar -->
     <xacro:property name="lidar_radius" value="0.035"/>
     <xacro:property name="lidar_thickness" value="0.024"/>
-    <xacro:property name="lidar_mass" value="0.19"/>
+    <xacro:property name="lidar_mass" value="0.100"/>
     <xacro:property name="lidar_color" value="blue"/>
     <xacro:property name="lidar_offset_z" value="0.046 "/>
-    <joint name="lidar_joint" type="fixed">
-        <parent link="chassis"/>
-        <child link="lidar_frame"/>
-        <xacro:if value="$(arg sim_mode)">
-            <origin xyz="0 0 ${chassis_thickness/2 + lidar_offset_z}" rpy="0 0 0"/>
-        </xacro:if>
-        <xacro:unless value="$(arg sim_mode)">
-            <origin xyz="0 0 ${chassis_thickness/2 + lidar_offset_z}" rpy="0 0 ${pi}"/>
-        </xacro:unless>
-    </joint>
-    <link name="lidar_frame">
-        <visual>
-            <geometry>
-                <cylinder radius="${lidar_radius}" length="${lidar_thickness}"/>
-            </geometry>
-            <material name="${lidar_color}"/>
-        </visual>
-        <collision>
-            <geometry>
-                <cylinder radius="${lidar_radius}" length="${lidar_thickness}"/>
-            </geometry>
-        </collision>
-        <xacro:inertial_cylinder mass="${lidar_mass}" radius="${lidar_radius}" length="${lidar_thickness}">
-            <origin xyz="0 0 0" rpy="0 0 0"/>
-        </xacro:inertial_cylinder>
-    </link>
-    <!-- BRACKET -->
     <xacro:property name="lidar_bracket_length" value="0.095"/>
     <xacro:property name="lidar_bracket_width" value="0.070"/>
     <xacro:property name="lidar_bracket_height" value="0.034"/>
-    <xacro:property name="lidar_bracket_mass" value="0.020"/>
+    <xacro:property name="lidar_bracket_mass" value="0.260"/>
     <xacro:property name="lidar_bracket_color" value="white"/>
-    <joint name="lidar_bracket_joint" type="fixed">
-        <parent link="chassis"/>
-        <child link="lidar_bracket"/>
-        <origin xyz="${-(lidar_bracket_length/2 - lidar_radius)} 0 ${chassis_thickness/2 + lidar_bracket_height/2}" rpy="0 0 0"/>
-    </joint>
-    <link name="lidar_bracket">
-        <visual>
-            <geometry>
-                <box size="${lidar_bracket_length} ${lidar_bracket_width} ${lidar_bracket_height}"/>
-            </geometry>
-            <material name="${lidar_bracket_color}"/>
-        </visual>
-        <collision>
-            <geometry>
-                <box size="${lidar_bracket_length} ${lidar_bracket_width} ${lidar_bracket_height}"/>
-            </geometry>
-        </collision>
-        <xacro:inertial_box mass="${lidar_bracket_mass}" x="${lidar_bracket_length}" y="${lidar_bracket_width}" z="${lidar_bracket_height}">
-            <origin xyz="0 0 0" rpy="0 0 0"/>
-        </xacro:inertial_box>
-    </link>
+    <xacro:arg name="test" default="true"/>
+    <!--  REAL ROBOT -->
+    <xacro:unless value="$(arg test)">
+        <!-- LIDAR -->
+        <joint name="lidar_joint" type="fixed">
+            <parent link="chassis"/>
+            <child link="lidar_frame"/>
+            <origin xyz="0 0 ${chassis_thickness/2 + lidar_offset_z}" rpy="0 0 ${pi}"/>
+        </joint>
+        <link name="lidar_frame">
+            <visual>
+                <origin xyz="0.013 0 -0.039" rpy="0 0 0"/>
+                <geometry>
+                    <mesh filename="package://vacuum_cleaner/description/mashes/RP-lidar-A1.stl" scale="0.001 0.001 0.001"/>
+                </geometry>
+                <material name="${lidar_color}"/>
+            </visual>
+            <collision>
+                <origin xyz="0.013 0 -0.039" rpy="0 0 0"/>
+                <geometry>
+                    <mesh filename="package://vacuum_cleaner/description/mashes/RP-lidar-A1.stl" scale="0.001 0.001 0.001"/>
+                </geometry>
+            </collision>
+            <xacro:inertial_cylinder mass="${lidar_mass}" radius="${lidar_radius}" length="${lidar_thickness}">
+                <origin xyz="0 0 0" rpy="0 0 0"/>
+            </xacro:inertial_cylinder>
+        </link>
+        <!-- BRACKET -->
+        <joint name="lidar_bracket_joint" type="fixed">
+            <parent link="chassis"/>
+            <child link="lidar_bracket"/>
+            <origin xyz="0 0 ${chassis_thickness/2}" rpy="0 0 0"/>
+        </joint>
+        <link name="lidar_bracket">
+            <visual>
+                <origin xyz="-0.0135 0 0" rpy="0 0 ${pi}"/>
+                <geometry>
+                    <mesh filename="package://vacuum_cleaner/description/mashes/Bracket.stl" scale="0.001 0.001 0.001"/>
+                </geometry>
+                <material name="${lidar_bracket_color}"/>
+            </visual>
+            <collision>
+                <origin xyz="-0.0135 0 0" rpy="0 0 ${pi}"/>
+                <geometry>
+                    <mesh filename="package://vacuum_cleaner/description/mashes/Bracket.stl" scale="0.001 0.001 0.001"/>
+                </geometry>
+            </collision>
+            <xacro:inertial_box mass="${lidar_bracket_mass}" x="${lidar_bracket_length}" y="${lidar_bracket_width}" z="${lidar_bracket_height}">
+                <origin xyz="-0.0135 0 ${lidar_bracket_height/2}" rpy="0 0 ${pi}"/>
+            </xacro:inertial_box>
+        </link>
+    </xacro:unless>
+    <!-- SIMULATION -->
+    <xacro:if value="$(arg test)">
+        <!-- LIDAR -->
+        <joint name="lidar_joint" type="fixed">
+            <parent link="chassis"/>
+            <child link="lidar_frame"/>
+            <origin xyz="0 0 ${chassis_thickness/2 + lidar_offset_z}" rpy="0 0 0"/>
+        </joint>
+        <link name="lidar_frame">
+            <visual>
+                <geometry>
+                    <cylinder radius="${lidar_radius}" length="${lidar_thickness}"/>
+                </geometry>
+                <material name="${lidar_color}"/>
+            </visual>
+            <collision>
+                <geometry>
+                    <cylinder radius="${lidar_radius}" length="${lidar_thickness}"/>
+                </geometry>
+            </collision>
+            <xacro:inertial_cylinder mass="${lidar_mass}" radius="${lidar_radius}" length="${lidar_thickness}">
+                <origin xyz="0 0 0" rpy="0 0 0"/>
+            </xacro:inertial_cylinder>
+        </link>
+        <!-- BRACKET -->
+        <joint name="lidar_bracket_joint" type="fixed">
+            <parent link="chassis"/>
+            <child link="lidar_bracket"/>
+            <origin xyz="${-(lidar_bracket_length/2 - lidar_radius)} 0 ${chassis_thickness/2 + lidar_bracket_height/2}" rpy="0 0 0"/>
+        </joint>
+        <link name="lidar_bracket">
+            <visual>
+                <geometry>
+                    <box size="${lidar_bracket_length} ${lidar_bracket_width} ${lidar_bracket_height}"/>
+                </geometry>
+                <material name="${lidar_bracket_color}"/>
+            </visual>
+            <collision>
+                <geometry>
+                    <box size="${lidar_bracket_length} ${lidar_bracket_width} ${lidar_bracket_height}"/>
+                </geometry>
+            </collision>
+            <xacro:inertial_box mass="${lidar_bracket_mass}" x="${lidar_bracket_length}" y="${lidar_bracket_width}" z="${lidar_bracket_height}">
+                <origin xyz="0 0 0" rpy="0 0 0"/>
+            </xacro:inertial_box>
+        </link>
+    </xacro:if>
 </robot>
