Commit message: adding gazebo colors

File: description/gazebo.xacro (robot description, xacro)
@@ -2,5 +2,5 @@
 <robot xmlns:xacro="http://www.ros.org/wiki/xacro">
     <xacro:if value="$(arg sim_mode)">
-        <!-- REFERENCES -->
+        <!-- GENERAL COLORS -->
         <gazebo reference="chassis">
             <material>Gazebo/White</material>
@@ -12,8 +12,14 @@
             <material>Gazebo/Blue</material>
         </gazebo>
+        <gazebo reference="caster_wheel_plate">
+            <material>Gazebo/Black</material>
+        </gazebo>
         <gazebo reference="caster_wheel">
             <material>Gazebo/Black</material>
             <mu1 value="0.001"/>
             <mu2 value="0.001"/>
+        </gazebo>
+        <gazebo reference="lidar_bracket">
+            <material>Gazebo/White</material>
         </gazebo>
         <!-- DISTANCE SENSORS -->
@@ -124,8 +130,4 @@
         </gazebo>
         <!-- right -->
-        <xacro:property name="right_vertical_min_angle" value="-0.2"/>
-        <xacro:property name="right_vertical_max_angle" value="0.2"/>
-        <xacro:property name="right_horizontal_min_angle" value="-1"/>
-        <xacro:property name="right_horizontal_max_angle" value="1"/>
         <gazebo reference="distance_sensor_right">
             <material>Gazebo/Black</material>

File: description/lidar.xacro (robot description, xacro)
@@ -36,8 +36,8 @@
     <joint name="lidar_bracket_joint" type="fixed">
         <parent link="chassis"/>
-        <child link="lidar_bracket_frame"/>
+        <child link="lidar_bracket"/>
         <origin xyz="${-(lidar_bracket_length/2 - lidar_radius)} 0 ${chassis_thickness/2 + lidar_bracket_height/2}" rpy="0 0 0"/>
     </joint>
-    <link name="lidar_bracket_frame">
+    <link name="lidar_bracket">
         <visual>
             <geometry>

Commit message: adding range sensors to hardware interface

File: description/gazebo.xacro (robot description, xacro)
@@ -23,5 +23,5 @@
             <material>Gazebo/White</material>
         </gazebo>
-        <!-- DISTANCE SENSORS -->
+        <!-- RANGE SENSORS -->
         <xacro:property name="horizontal_samples" value="10"/>
         <xacro:property name="horizontal_resolution" value="1"/>
@@ -39,9 +39,54 @@
         <xacro:property name="right_vertical_min_angle" value="-0.2"/>
         <xacro:property name="right_vertical_max_angle" value="0.2"/>
+        <!-- left -->
+        <gazebo reference="range_sensor_left">
+            <material>Gazebo/Black</material>
+            <pose>0 0 0 0 0 0</pose>
+            <sensor name="range_sensor_left" type="ray">
+                <always_on>true</always_on>
+                <visualize>true</visualize>
+                <update_rate>30</update_rate>
+                <ray>
+                    <scan>
+                        <horizontal>
+                            <samples>${horizontal_samples}</samples>
+                            <resolution>${horizontal_resolution}</resolution>
+                            <min_angle>${horizontal_min_angle}</min_angle>
+                            <max_angle>${horizontal_max_angle}</max_angle>
+                        </horizontal>
+                        <vertical>
+                            <samples>${vertical_samples}</samples>
+                            <resolution>${vertical_resolution}</resolution>
+                            <min_angle>${left_vertical_min_angle}</min_angle>
+                            <max_angle>${left_vertical_max_angle}</max_angle>
+                        </vertical>
+                    </scan>
+                    <range>
+                        <min>${range_min}</min>
+                        <max>${range_max}</max>
+                        <resolution>${range_resolution}</resolution>
+                    </range>
+                    <noise>
+                        <type>gaussian</type>
+                        <mean>0.0</mean>
+                        <stddev>0.01</stddev>
+                    </noise>
+                </ray>
+                <plugin name="range_sensor_left" filename="libgazebo_ros_ray_sensor.so">
+                    <ros>
+                        <namespace>/range_sensor_broadcaster_left</namespace>
+                        <remapping>~/out:=range</remapping>
+                    </ros>
+                    <output_type>sensor_msgs/Range</output_type>
+                    <radiation_type>infrared</radiation_type>
+                    <frame_name>range_sensor_left</frame_name>
+                </plugin>
+            </sensor>
+        </gazebo>
         <!-- front -->
-        <gazebo reference="distance_sensor_front">
+        <gazebo reference="range_sensor_front">
             <material>Gazebo/Black</material>
             <pose>0 0 0 0 0 0</pose>
-            <sensor name="range_sensor_frotn" type="ray">
+            <sensor name="range_sensor_front" type="ray">
                 <always_on>true</always_on>
                 <visualize>true</visualize>
@@ -75,60 +120,15 @@
                 <plugin name="range_sensor_front" filename="libgazebo_ros_ray_sensor.so">
                     <ros>
-                        <namespace>/bumper/distance</namespace>
-                        <remapping>~/out:=front</remapping>
+                        <namespace>range_sensor_broadcaster_front</namespace>
+                        <remapping>~/out:=range</remapping>
                     </ros>
                     <output_type>sensor_msgs/Range</output_type>
                     <radiation_type>infrared</radiation_type>
-                    <frame_name>distance_sensor_front</frame_name>
-                </plugin>
-            </sensor>
-        </gazebo>
-        <!-- left -->
-        <gazebo reference="distance_sensor_left">
-            <material>Gazebo/Black</material>
-            <pose>0 0 0 0 0 0</pose>
-            <sensor name="range_sensor_left" type="ray">
-                <always_on>true</always_on>
-                <visualize>true</visualize>
-                <update_rate>30</update_rate>
-                <ray>
-                    <scan>
-                        <horizontal>
-                            <samples>${horizontal_samples}</samples>
-                            <resolution>${horizontal_resolution}</resolution>
-                            <min_angle>${horizontal_min_angle}</min_angle>
-                            <max_angle>${horizontal_max_angle}</max_angle>
-                        </horizontal>
-                        <vertical>
-                            <samples>${vertical_samples}</samples>
-                            <resolution>${vertical_resolution}</resolution>
-                            <min_angle>${left_vertical_min_angle}</min_angle>
-                            <max_angle>${left_vertical_max_angle}</max_angle>
-                        </vertical>
-                    </scan>
-                    <range>
-                        <min>${range_min}</min>
-                        <max>${range_max}</max>
-                        <resolution>${range_resolution}</resolution>
-                    </range>
-                    <noise>
-                        <type>gaussian</type>
-                        <mean>0.0</mean>
-                        <stddev>0.01</stddev>
-                    </noise>
-                </ray>
-                <plugin name="range_sensor_left" filename="libgazebo_ros_ray_sensor.so">
-                    <ros>
-                        <namespace>/bumper/distance</namespace>
-                        <remapping>~/out:=left</remapping>
-                    </ros>
-                    <output_type>sensor_msgs/Range</output_type>
-                    <radiation_type>infrared</radiation_type>
-                    <frame_name>distance_sensor_left</frame_name>
+                    <frame_name>range_sensor_front</frame_name>
                 </plugin>
             </sensor>
         </gazebo>
         <!-- right -->
-        <gazebo reference="distance_sensor_right">
+        <gazebo reference="range_sensor_right">
             <material>Gazebo/Black</material>
             <pose>0 0 0 0 0 0</pose>
@@ -165,10 +165,10 @@
                 <plugin name="range_sensor_right" filename="libgazebo_ros_ray_sensor.so">
                     <ros>
-                        <namespace>/bumper/distance</namespace>
-                        <remapping>~/out:=right</remapping>
+                        <namespace>range_sensor_broadcaster_right</namespace>
+                        <remapping>~/out:=range</remapping>
                     </ros>
                     <output_type>sensor_msgs/Range</output_type>
                     <radiation_type>infrared</radiation_type>
-                    <frame_name>distance_sensor_right</frame_name>
+                    <frame_name>range_sensor_right</frame_name>
                 </plugin>
             </sensor>

File: description/robot.urdf.xacro (robot description, xacro)
@@ -7,5 +7,5 @@
     <xacro:include filename="materials.xacro"/>
     <xacro:include filename="robot_core.xacro"/>
-    <xacro:include filename="bumper_distance_sensors.xacro"/>
+    <xacro:include filename="range_sensors.xacro"/>
     <xacro:include filename="lidar.xacro"/>
     <xacro:include filename="ros2_control.xacro"/>

File: description/ros2_control.xacro (robot description, xacro)
@@ -8,9 +8,15 @@
         <param name="left_wheel_name">left_wheel_joint</param>
         <param name="right_wheel_name">right_wheel_joint</param>
-        <param name="serial_device">/dev/serial/by-id/usb-Arduino_RaspberryPi_Pico_644861E6228B85D3-if00</param>
-        <param name="baud_rate">115200</param>
-        <param name="timeout_ms">1000</param>
         <param name="enc_counts_per_rev">575</param>
         <param name="wheel_radius_mm">32</param>
+        <param name="motors_port">/dev/serial/by-id/usb-Arduino_RaspberryPi_Pico_644861E6228B85D3-if00</param>
+        <param name="motors_baud_rate">115200</param>
+        <param name="motors_timeout_ms">1000</param>
+        <param name="sensors_port">/dev/serial/by-id/usb-Arduino_RaspberryPi_Pico_304C61E62BB46493-if00</param>
+        <param name="sensors_baud_rate">115200</param>
+        <param name="sensors_timeout_ms">1000</param>
+        <param name="range_sensor_left_name">range_sensor_left</param>
+        <param name="range_sensor_front_name">range_sensor_front</param>
+        <param name="range_sensor_right_name">range_sensor_right</param>
       </hardware>
       <joint name="left_wheel_joint">
@@ -24,4 +30,16 @@
         <state_interface name="velocity"/>
       </joint>
+      <sensor name="range_sensor_left">
+        <state_interface name="range"/>
+        <param name="frame_id">range_sensor_left</param>
+      </sensor>
+      <sensor name="range_sensor_front">
+        <state_interface name="range"/>
+        <param name="frame_id">range_sensor_front</param>
+      </sensor>
+      <sensor name="range_sensor_right">
+        <state_interface name="range"/>
+        <param name="frame_id">range_sensor_right</param>
+      </sensor>
     </ros2_control>
   </xacro:unless>
@@ -29,23 +47,23 @@
   <xacro:if value="$(arg sim_mode)">
     <ros2_control name="GazeboSystem" type="system">
-        <hardware>
-            <plugin>gazebo_ros2_control/GazeboSystem</plugin>
-        </hardware>
-        <joint name="left_wheel_joint">
-            <command_interface name="velocity">
-                <param name="min">-10</param>
-                <param name="max">10</param>
-            </command_interface>
-            <state_interface name="velocity"/>
-            <state_interface name="position"/>
-        </joint>
-        <joint name="right_wheel_joint">
-            <command_interface name="velocity">
-                <param name="min">-10</param>
-                <param name="max">10</param>
-            </command_interface>
-            <state_interface name="velocity"/>
-            <state_interface name="position"/>
-        </joint>
+      <hardware>
+          <plugin>gazebo_ros2_control/GazeboSystem</plugin>
+      </hardware>
+      <joint name="left_wheel_joint">
+          <command_interface name="velocity">
+              <param name="min">-10</param>
+              <param name="max">10</param>
+          </command_interface>
+          <state_interface name="velocity"/>
+          <state_interface name="position"/>
+      </joint>
+      <joint name="right_wheel_joint">
+          <command_interface name="velocity">
+              <param name="min">-10</param>
+              <param name="max">10</param>
+          </command_interface>
+          <state_interface name="velocity"/>
+          <state_interface name="position"/>
+      </joint>
     </ros2_control>
   </xacro:if>

Commit message: changing wheel names

File: description/gazebo.xacro (robot description, xacro)
@@ -6,8 +6,8 @@
             <material>Gazebo/White</material>
         </gazebo>
-        <gazebo reference="left_wheel">
+        <gazebo reference="wheel_left">
             <material>Gazebo/Blue</material>
         </gazebo>
-        <gazebo reference="right_wheel">
+        <gazebo reference="wheel_right">
             <material>Gazebo/Blue</material>
         </gazebo>

File: description/robot_core.xacro (robot description, xacro)
@@ -48,11 +48,11 @@
     <xacro:property name="wheel_offset_x" value="0"/>
     <xacro:property name="wheel_separation" value="0.231"/>
-    <joint name="left_wheel_joint" type="continuous">
+    <joint name="wheel_left_joint" type="continuous">
         <parent link="base_link"/>
-        <child link="left_wheel"/>
+        <child link="wheel_left"/>
         <origin xyz="${wheel_offset_x} ${wheel_separation/2} ${wheel_radius}" rpy="-${pi/2} 0 0" />
         <axis xyz="0 0 1"/>
     </joint>
-    <link name="left_wheel">
+    <link name="wheel_left">
         <visual>
             <geometry>
@@ -71,11 +71,11 @@
     </link>
     <!-- RIGHT WHEEL LINK -->
-    <joint name="right_wheel_joint" type="continuous">
+    <joint name="wheel_right_joint" type="continuous">
         <parent link="base_link"/>
-        <child link="right_wheel"/>
+        <child link="wheel_right"/>
         <origin xyz="${wheel_offset_x} ${-wheel_separation/2} ${wheel_radius}" rpy="${pi/2} 0 0" />
         <axis xyz="0 0 -1"/>
     </joint>
-    <link name="right_wheel">
+    <link name="wheel_right">
         <visual>
             <geometry>

File: description/ros2_control.xacro (robot description, xacro)
@@ -7,10 +7,10 @@
         <plugin>vacuum_cleaner/VacuumCleanerHardware</plugin>
       </hardware>
-      <joint name="left_wheel_joint">
+      <joint name="wheel_left_joint">
         <command_interface name="velocity"/>
         <state_interface name="position"/>
         <state_interface name="velocity"/>
       </joint>
-      <joint name="right_wheel_joint">
+      <joint name="wheel_right_joint">
         <command_interface name="velocity"/>
         <state_interface name="position"/>
@@ -67,5 +67,5 @@
         <plugin>gazebo_ros2_control/GazeboSystem</plugin>
       </hardware>
-      <joint name="left_wheel_joint">
+      <joint name="wheel_left_joint">
         <command_interface name="velocity">
           <param name="min">-10</param>
@@ -75,5 +75,5 @@
         <state_interface name="position"/>
       </joint>
-      <joint name="right_wheel_joint">
+      <joint name="wheel_right_joint">
         <command_interface name="velocity">
           <param name="min">-10</param>

Commit message: updating URDF

File: description/gazebo.xacro (robot description, xacro)
@@ -7,19 +7,31 @@
         </gazebo>
         <gazebo reference="wheel_left">
+            <material>Gazebo/Black</material>
+        </gazebo>
+        <gazebo reference="wheel_right">
+            <material>Gazebo/Black</material>
+        </gazebo>
+        <gazebo reference="sweeper_left">
+            <material>Gazebo/Black</material>
+        </gazebo>
+        <gazebo reference="sweeper_right">
+            <material>Gazebo/Black</material>
+        </gazebo>
+        <gazebo reference="caster_wheel_plate">
+            <material>Gazebo/Black</material>
+        </gazebo>
+        <gazebo reference="caster_wheel">
             <material>Gazebo/Blue</material>
-        </gazebo>
-        <gazebo reference="wheel_right">
-            <material>Gazebo/Blue</material>
-        </gazebo>
-        <gazebo reference="caster_wheel_plate">
-            <material>Gazebo/Black</material>
-        </gazebo>
-        <gazebo reference="caster_wheel">
-            <material>Gazebo/Black</material>
             <mu1 value="0.001"/>
             <mu2 value="0.001"/>
         </gazebo>
+        <gazebo reference="frame_bracket">
+            <material>Gazebo/Blue</material>
+        </gazebo>
         <gazebo reference="lidar_bracket">
             <material>Gazebo/White</material>
+        </gazebo>
+        <gazebo reference="raspberry_pi">
+            <material>Gazebo/Black</material>
         </gazebo>
         <!-- RANGE SENSORS -->

File: description/robot.urdf.xacro (robot description, xacro)
@@ -10,4 +10,5 @@
     <xacro:include filename="range_sensors.xacro"/>
     <xacro:include filename="lidar.xacro"/>
+    <xacro:include filename="raspberry_pi.xacro"/>
     <xacro:include filename="ros2_control.xacro"/>
     <xacro:include filename="gazebo.xacro"/>

File: description/robot_core.xacro (robot description, xacro)
@@ -15,5 +15,5 @@
     <xacro:property name="chassis_radius" value="0.150"/>
     <xacro:property name="chassis_thickness" value="0.065"/>
-    <xacro:property name="chassis_mass" value="0.500"/>
+    <xacro:property name="chassis_mass" value="2.000"/>
     <xacro:property name="chassis_color" value="white"/>
     <xacro:property name="chassis_offset_z" value="0.0425"/>
@@ -38,5 +38,5 @@
         </collision>
         <xacro:inertial_cylinder mass="${chassis_mass}" radius="${chassis_radius}" length="${chassis_thickness}">
-            <origin xyz="0 0 0" rpy="0 0 0"/>
+            <origin xyz="0.01 0 0" rpy="0 0 0"/>
         </xacro:inertial_cylinder>
     </link>
@@ -44,6 +44,6 @@
     <xacro:property name="wheel_radius" value="0.0325"/>
     <xacro:property name="wheel_thickness" value="0.015"/>
-    <xacro:property name="wheel_mass" value="0.050"/>
-    <xacro:property name="wheel_color" value="blue"/>
+    <xacro:property name="wheel_mass" value="0.030"/>
+    <xacro:property name="wheel_color" value="black"/>
     <xacro:property name="wheel_offset_x" value="0"/>
     <xacro:property name="wheel_separation" value="0.231"/>
@@ -96,5 +96,5 @@
     <xacro:property name="caster_wheel_plate_radius" value="0.025"/>
     <xacro:property name="caster_wheel_plate_thickness" value="0.0001"/>
-    <xacro:property name="caster_wheel_plate_mass" value="0.010"/>
+    <xacro:property name="caster_wheel_plate_mass" value="0.005"/>
     <xacro:property name="caster_wheel_plate_color" value="blue"/>
     <xacro:property name="caster_wheel_plate_offset_x" value="0.1"/>
@@ -125,5 +125,5 @@
     <xacro:property name="caster_wheel_radius" value="0.010"/>
     <xacro:property name="caster_wheel_thickness" value="0.020"/>
-    <xacro:property name="caster_wheel_mass" value="0.020"/>
+    <xacro:property name="caster_wheel_mass" value="0.015"/>
     <xacro:property name="caster_wheel_color" value="blue"/>
     <xacro:property name="caster_wheel_offset_x" value="0.008"/>
@@ -146,5 +146,5 @@
             </geometry>
         </collision>
-        <xacro:inertial_cylinder mass="0.1" radius="${caster_wheel_radius}" length="${caster_wheel_thickness}">
+        <xacro:inertial_cylinder mass="${caster_wheel_mass}" radius="${caster_wheel_radius}" length="${caster_wheel_thickness}">
             <origin xyz="0 0 0" rpy="0 0 0"/>
         </xacro:inertial_cylinder>
