Commit message: adjusting range sensor angles

File: description/gazebo.xacro (robot description, xacro)
@@ -38,17 +38,17 @@
         <xacro:property name="horizontal_samples" value="10"/>
         <xacro:property name="horizontal_resolution" value="1"/>
-        <xacro:property name="horizontal_min_angle" value="-1"/>
-        <xacro:property name="horizontal_max_angle" value="1"/>
         <xacro:property name="vertical_samples" value="10"/>
         <xacro:property name="vertical_resolution" value="1"/>
+        <xacro:property name="vertical_min_angle" value="-0.4"/>
+        <xacro:property name="vertical_max_angle" value="0.4"/>
         <xacro:property name="range_min" value="0.001"/>
         <xacro:property name="range_max" value="0.07"/>
         <xacro:property name="range_resolution" value="0.01"/>
-        <xacro:property name="front_vertical_min_angle" value="-0.3"/>
-        <xacro:property name="front_vertical_max_angle" value="0.3"/>
-        <xacro:property name="left_vertical_min_angle" value="-0.2"/>
-        <xacro:property name="left_vertical_max_angle" value="0.2"/>
-        <xacro:property name="right_vertical_min_angle" value="-0.2"/>
-        <xacro:property name="right_vertical_max_angle" value="0.2"/>
+        <xacro:property name="left_horizontal_min_angle" value="-0.8"/>
+        <xacro:property name="left_horizontal_max_angle" value="1.2"/>
+        <xacro:property name="front_horizontal_min_angle" value="-1.2"/>
+        <xacro:property name="front_horizontal_max_angle" value="1.2"/>
+        <xacro:property name="right_horizontal_min_angle" value="-1.2"/>
+        <xacro:property name="right_horizontal_max_angle" value="0.8"/>
         <!-- left -->
         <gazebo reference="range_sensor_left">
@@ -64,12 +64,12 @@
                             <samples>${horizontal_samples}</samples>
                             <resolution>${horizontal_resolution}</resolution>
-                            <min_angle>${horizontal_min_angle}</min_angle>
-                            <max_angle>${horizontal_max_angle}</max_angle>
+                            <min_angle>${left_horizontal_min_angle}</min_angle>
+                            <max_angle>${left_horizontal_max_angle}</max_angle>
                         </horizontal>
                         <vertical>
                             <samples>${vertical_samples}</samples>
                             <resolution>${vertical_resolution}</resolution>
-                            <min_angle>${left_vertical_min_angle}</min_angle>
-                            <max_angle>${left_vertical_max_angle}</max_angle>
+                            <min_angle>${vertical_min_angle}</min_angle>
+                            <max_angle>${vertical_max_angle}</max_angle>
                         </vertical>
                     </scan>
@@ -109,12 +109,12 @@
                             <samples>${horizontal_samples}</samples>
                             <resolution>${horizontal_resolution}</resolution>
-                            <min_angle>${horizontal_min_angle}</min_angle>
-                            <max_angle>${horizontal_max_angle}</max_angle>
+                            <min_angle>${front_horizontal_min_angle}</min_angle>
+                            <max_angle>${front_horizontal_max_angle}</max_angle>
                         </horizontal>
                         <vertical>
                             <samples>${vertical_samples}</samples>
                             <resolution>${vertical_resolution}</resolution>
-                            <min_angle>${front_vertical_min_angle}</min_angle>
-                            <max_angle>${front_vertical_max_angle}</max_angle>
+                            <min_angle>${vertical_min_angle}</min_angle>
+                            <max_angle>${vertical_max_angle}</max_angle>
                         </vertical>
                     </scan>
@@ -154,12 +154,12 @@
                             <samples>${horizontal_samples}</samples>
                             <resolution>${horizontal_resolution}</resolution>
-                            <min_angle>${horizontal_min_angle}</min_angle>
-                            <max_angle>${horizontal_max_angle}</max_angle>
+                            <min_angle>${right_horizontal_min_angle}</min_angle>
+                            <max_angle>${right_horizontal_max_angle}</max_angle>
                         </horizontal>
                         <vertical>
                             <samples>${vertical_samples}</samples>
                             <resolution>${vertical_resolution}</resolution>
-                            <min_angle>${right_vertical_min_angle}</min_angle>
-                            <max_angle>${right_vertical_max_angle}</max_angle>
+                            <min_angle>${vertical_min_angle}</min_angle>
+                            <max_angle>${vertical_max_angle}</max_angle>
                         </vertical>
                     </scan>

Commit message: changing settings for lidar sensor

File: description/gazebo.xacro (robot description, xacro)
@@ -203,5 +203,5 @@
                     <range>
                         <min>0.15</min>
-                        <max>6</max>
+                        <max>12</max>
                     </range>
                 </ray>

File: description/lidar.xacro (robot description, xacro)
@@ -3,5 +3,5 @@
     <xacro:property name="lidar_radius" value="0.035"/>
     <xacro:property name="lidar_thickness" value="0.024"/>
-    <xacro:property name="lidar_mass" value="0.100"/>
+    <xacro:property name="lidar_mass" value="0.170"/>
     <xacro:property name="lidar_color" value="blue"/>
     <xacro:property name="lidar_offset_z" value="0.046 "/>
